Commit message: craeate arm and spawn in gazebo

File: ROS2_for_Beginners_Level2_TF_URDF_RVIZ_GAZEBO/install/my_robot_description/share/my_robot_description/urdf/common_properties.xacro (robot description, xacro)
@@ -9,4 +9,10 @@
     <material name="grey">
         <color rgba="0.5 0.5 0.5 1" />
+    </material>
+    <material name="black">
+        <color rgba="0 0 0 1" />
+    </material>
+    <material name="red">
+        <color rgba="1 0 0 1" />
     </material>
     <xacro:macro name="box_inertia" params="m x y z o_xyz o_rpy">
