Commit message: concatinate both arm and mobile robot and finish the project.

File: ROS2_for_Beginners_Level2_TF_URDF_RVIZ_GAZEBO/install/my_robot_description/share/my_robot_description/urdf/arm.xacro (robot description, xacro)
@@ -11,5 +11,5 @@
     <xacro:property name="hand_length" value="0.3" />
     <xacro:property name="hand_mass" value="0.3"/>
-    <link name="base_footprint" />
+    <!-- <link name="base_footprint" /> -->
     <link name="arm_base_link">
         <visual>
@@ -60,9 +60,9 @@
         <xacro:cylinder_inertia m="${hand_mass}" radius="${hand_radius}" height="${hand_length}" o_xyz="0 0 ${hand_length / 2.0}" o_rpy="0 0 0" />
     </link>
-    <joint name="base_joint" type="fixed">
+    <!-- <joint name="base_joint" type="fixed">
         <parent link="base_footprint" />
         <child link="arm_base_link" />
         <origin xyz="0 0 0" rpy="0 0 0" />
-    </joint>
+    </joint> -->
     <joint name="arm_base_forearm_joint" type="revolute">
         <parent link="arm_base_link" />

File: ROS2_for_Beginners_Level2_TF_URDF_RVIZ_GAZEBO/install/my_robot_description/share/my_robot_description/urdf/mobile_robot.urdf.xacro (robot description, xacro)
@@ -4,4 +4,11 @@
     <xacro:include filename="mobile_base.xacro" />
     <xacro:include filename="my_robot_gazebo.xacro" />
+    <xacro:include filename="arm.xacro"/>
+    <xacro:include filename="arm_gazebo.xacro"/>
     <xacro:include filename="camera.xacro" />
+    <joint name="mobile_base_arm_base_joint" type="fixed">
+        <parent link="base_link"/>
+        <child link="arm_base_link"/>
+        <origin xyz="${base_length / 4.0} 0 ${base_height}" rpy="0 0 0"/>
+    </joint>
 </robot>
